Commit message: add rqt dos testes de sexta

File: bill_ws/install/bill/share/bill/description/gazebo_control.xacro (robot description, xacro)
@@ -28,5 +28,5 @@
         <max_wheel_acceleration>10.0</max_wheel_acceleration>
         <!-- Frames -->
-        <odometry_frame>odom</odometry_frame>
+        <odometry_frame>odometry</odometry_frame>
         <robot_base_frame>base_link</robot_base_frame>
         <!-- Output -->

File: bill_ws/install/bill/share/bill/description/lidar.xacro (robot description, xacro)
@@ -39,6 +39,6 @@
                 </scan>
                 <range>
-                    <min>0.1</min>
-                    <max>25</max>
+                    <min>0.02</min>
+                    <max>12</max>
                 </range>
             </ray>

File: bill_ws/install/bill/share/bill/description/robot_core.xacro (robot description, xacro)
@@ -116,6 +116,6 @@
         <parent link="base_link"/>
         <child link="rear_left_wheel"/>
-        <origin xyz="${-wheel_offset_x} ${wheel_offset_y} 0" rpy="-${pi/2} 0 0" />
-        <axis xyz="0 0 1"/>
+        <origin xyz="${-wheel_offset_x} ${-wheel_offset_y} 0" rpy="-${pi/2} 0 0" />
+        <axis xyz="0 0 -1"/>
     </joint>
     <transmission name="rear_left_wheel_trans">
@@ -148,6 +148,6 @@
         <parent link="base_link"/>
         <child link="rear_right_wheel"/>
-        <origin xyz="${-wheel_offset_x} ${-wheel_offset_y} 0" rpy="${pi/2} 0 0" />
-        <axis xyz="0 0 -1"/>
+        <origin xyz="${-wheel_offset_x} ${wheel_offset_y} 0" rpy="${pi/2} 0 0" />
+        <axis xyz="0 0 1"/>
     </joint>
     <transmission name="rear_right_wheel_trans">

Commit message: commit

File: bill_ws/install/bill/share/bill/description/gazebo_control.xacro (robot description, xacro)
@@ -28,5 +28,5 @@
         <max_wheel_acceleration>10.0</max_wheel_acceleration>
         <!-- Frames -->
-        <odometry_frame>odometry</odometry_frame>
+        <odometry_frame>odom</odometry_frame>
         <robot_base_frame>base_link</robot_base_frame>
         <!-- Output -->

File: bill_ws/install/bill/share/bill/description/lidar.xacro (robot description, xacro)
@@ -34,6 +34,6 @@
                     <horizontal>
                         <samples>160</samples>
-                        <min_angle>-1.4</min_angle> <!-- Ângulo de -80º -->
-                        <max_angle>1.4</max_angle>  <!-- Ângulo de 80º -->
+                        <min_angle>-1.59</min_angle> <!-- Ângulo de -80º -->
+                        <max_angle>1.59</max_angle>  <!-- Ângulo de 80º -->
                     </horizontal>
                 </scan>

File: bill_ws/install/bill/share/bill/description/robot.urdf.xacro (robot description, xacro)
@@ -3,5 +3,5 @@
 	<!--<xacro:include filename="robot_core_lr.xacro"/>-->
 	<xacro:include filename="robot_core.xacro"/>
-	<!-- <xacro:include filename="gazebo_control.xacro"/> -->
+	<xacro:include filename="gazebo_control.xacro"/>
 	<xacro:include filename="lidar.xacro"/>
 	<xacro:include filename="ros2_control.xacro"/>

File: bill_ws/install/bill/share/bill/description/robot_core.xacro (robot description, xacro)
@@ -5,7 +5,7 @@
     <xacro:include filename="common.xacro"/>
     <!-- Robot Variables -->
-    <xacro:property name="chassis_length" value="0.6"/>
-    <xacro:property name="chassis_width" value="0.4"/>
-    <xacro:property name="chassis_height" value="1.2"/>
+    <xacro:property name="chassis_length" value="0.5"/>
+    <xacro:property name="chassis_width" value="0.3"/>
+    <xacro:property name="chassis_height" value="1.17"/>
     <xacro:property name="chassis_mass" value="22.2"/>
     <xacro:property name="wheel_radius" value="0.07"/>
@@ -116,6 +116,6 @@
         <parent link="base_link"/>
         <child link="rear_left_wheel"/>
-        <origin xyz="${-wheel_offset_x} ${-wheel_offset_y} 0" rpy="-${pi/2} 0 0" />
-        <axis xyz="0 0 -1"/>
+        <origin xyz="${-wheel_offset_x} ${wheel_offset_y} 0" rpy="-${pi/2} 0 0" />
+        <axis xyz="0 0 1"/>
     </joint>
     <transmission name="rear_left_wheel_trans">
@@ -148,6 +148,6 @@
         <parent link="base_link"/>
         <child link="rear_right_wheel"/>
-        <origin xyz="${-wheel_offset_x} ${wheel_offset_y} 0" rpy="${pi/2} 0 0" />
-        <axis xyz="0 0 1"/>
+        <origin xyz="${-wheel_offset_x} ${-wheel_offset_y} 0" rpy="${pi/2} 0 0" />
+        <axis xyz="0 0 -1"/>
     </joint>
     <transmission name="rear_right_wheel_trans">
