Commit message: add bill simulado ainda não funciona 100% precisa de correção na física do robô

File: bill_ws/install/bill/share/bill/description/common.xacro (robot description, xacro)
@@ -1,60 +1 @@
-<?xml version="1.0"?>
-<robot xmlns:xacro="http://www.ros.org/wiki/xacro" >
-    <!-- This file contains the macros used across the URDF files -->
-    <!-- Inertial Macros -->
-    <!-- Inertial Sphere Macros -->
-    <xacro:macro name="inertial_sphere" params="mass radius *origin">
-        <inertial>
-            <xacro:insert_block name="origin"/>
-            <mass value="${mass}" />
-            <inertia ixx="${(2/5) * mass * (radius*radius)}" ixy="0.0" ixz="0.0"
-                    iyy="${(2/5) * mass * (radius*radius)}" iyz="0.0"
-                    izz="${(2/5) * mass * (radius*radius)}" />
-        </inertial>
-    </xacro:macro>
-    <!-- Inertial Box Macros -->
-    <xacro:macro name="inertial_box" params="mass x y z *origin">
-        <inertial>
-            <xacro:insert_block name="origin"/>
-            <mass value="${mass}" />
-            <inertia ixx="${(1/12) * mass * (y*y+z*z)}" ixy="0.0" ixz="0.0"
-                    iyy="${(1/12) * mass * (x*x+z*z)}" iyz="0.0"
-                    izz="${(1/12) * mass * (x*x+y*y)}" />
-        </inertial>
-    </xacro:macro>
-    <!-- Inertial Cylinder Macros -->
-    <xacro:macro name="inertial_cylinder" params="mass length radius *origin">
-        <inertial>
-            <xacro:insert_block name="origin"/>
-            <mass value="${mass}" />
-            <inertia ixx="${(1/12) * mass * (3*radius*radius + length*length)}" ixy="0.0" ixz="0.0"
-                    iyy="${(1/12) * mass * (3*radius*radius + length*length)}" iyz="0.0"
-                    izz="${(1/2) * mass * (radius*radius)}" />
-        </inertial>
-    </xacro:macro>
-    <!-- Material Macros -->
-    <material name="white">
-        <color rgba="1 1 1 1" />
-    </material>
-    <material name="orange">
-        <color rgba="1 0.3 0.1 1"/>
-    </material>
-    <material name="blue">
-        <color rgba="0.2 0.2 1 1"/>
-    </material>
-    <material name="black">
-        <color rgba="0 0 0 1"/>
-    </material>
-    <material name="red">
-        <color rgba="1 0 0 1"/>
-    </material>
-    <material name="grey">
-        <color rgba="0.631 0.631 0.631 1"/>
-    </material>
-    <material name="purple">
-        <color rgba="0.78 0.153 0.71 1"/>
-    </material>
-    <material name="green">
-        <color rgba="0.149 0.612 0.082 1"/>
-    </material>
-</robot>
+/home/vfran/billeagle_ws/bill_ws/src/bill/description/common.xacro

File: bill_ws/install/bill/share/bill/description/gazebo_control.xacro (robot description, xacro)
@@ -1,38 +1 @@
-<?xml version="1.0"?>
-<robot xmlns:xacro="http://www.ros.org/wiki/xacro">
-    <xacro:property name="wheel_radius" value="0.07"/>
-    <xacro:property name="wheel_thickness" value="0.05"/>
-    <xacro:property name="wheel_mass" value="0.2"/>
-    <xacro:property name="wheel_offset_x" value="0.2"/>
-    <xacro:property name="wheel_offset_y" value="${chassis_width/2 + wheel_thickness/2}"/>
-    <xacro:property name="wheel_offset_z" value="0.0"/>
-    <!-- Gazebo plugin for 4-wheel drive robots -->
-   <gazebo>
-      <plugin name="differential_drive_controller" filename="libgazebo_ros_diff_drive.so">
-        <!-- <ros>
-          <remapping>odom:=odom/unfiltered</remapping>
-        </ros> -->
-        <!-- <updateRate>100</updateRate> -->
-        <!-- Wheel Info -->
-        <num_wheel_pairs>2</num_wheel_pairs>
-        <left_joint>front_left_wheel_joint</left_joint>
-        <right_joint>front_right_wheel_joint</right_joint>
-        <left_joint>rear_left_wheel_joint</left_joint>
-        <right_joint>rear_right_wheel_joint</right_joint>
-        <wheel_separation>${wheel_offset_y*2}</wheel_separation>
-        <wheel_separation>${wheel_offset_y*2}</wheel_separation>
-        <wheel_diameter>${wheel_radius*2}</wheel_diameter>
-        <wheel_diameter>${wheel_radius*2}</wheel_diameter>
-        <!-- Limits -->
-        <max_wheel_torque>200</max_wheel_torque>
-        <max_wheel_acceleration>10.0</max_wheel_acceleration>
-        <!-- Frames -->
-        <odometry_frame>odom</odometry_frame>
-        <robot_base_frame>base_link</robot_base_frame>
-        <!-- Output -->
-        <publish_odom>true</publish_odom>
-        <publish_odom_tf>true</publish_odom_tf>
-        <publish_wheel_tf>true</publish_wheel_tf>
-      </plugin>
-    </gazebo>
-</robot>
+/home/vfran/billeagle_ws/bill_ws/src/bill/description/gazebo_control.xacro

File: bill_ws/install/bill/share/bill/description/lidar.xacro (robot description, xacro)
@@ -1,54 +1 @@
-<?xml version="1.0"?>
-<robot xmlns:xacro="http://www.ros.org/wiki/xacro" >
-    <!-- Lidar's urdf-->
-    <joint name="laser_joint" type="fixed">
-        <parent link="chassis_link"/>
-        <child link="laser_link"/>
-        <origin xyz="0.3 0 0.3" rpy="0 0 0"/>
-    </joint>
-    <link name="laser_link">
-        <visual>
-            <geometry>
-                <cylinder radius="0.05" length="0.05"/>
-            </geometry>
-            <material name="black"/>
-        </visual>
-        <collision>
-            <geometry>
-                <cylinder radius="0.05" length="0.05"/>
-            </geometry>
-        </collision>
-        <xacro:inertial_cylinder mass="0.1" length="0.05" radius="0.05">
-            <origin xyz="0 0 0" rpy="0 0 0"/>
-        </xacro:inertial_cylinder>
-    </link>
-    <!-- 2D Lidar Gazebo Sensor Plugin  -->
-    <gazebo reference="laser_link">
-        <material>Gazebo/Black</material>
-        <sensor name="laser" type="ray">
-            <pose> 0 0 0 0 0 0 </pose>
-            <visualize>true</visualize>
-            <update_rate>10</update_rate>
-            <ray>
-                <scan>
-                    <horizontal>
-                        <samples>160</samples>
-                        <min_angle>-1.59</min_angle> <!-- Ângulo de -80º -->
-                        <max_angle>1.59</max_angle>  <!-- Ângulo de 80º -->
-                    </horizontal>
-                </scan>
-                <range>
-                    <min>0.02</min>
-                    <max>12</max>
-                </range>
-            </ray>
-            <plugin name="laser_controller" filename="libgazebo_ros_ray_sensor.so">
-                <ros>
-                    <argument>--ros-args --remap ~/out:=scan_gazebo</argument>
-                </ros>
-                <output_type>sensor_msgs/LaserScan</output_type>
-                <frame_name>laser_link</frame_name>
-            </plugin>
-        </sensor>
-    </gazebo>
-</robot>
+/home/vfran/billeagle_ws/bill_ws/src/bill/description/lidar.xacro

File: bill_ws/install/bill/share/bill/description/robot.urdf.xacro (robot description, xacro)
@@ -1,8 +1 @@
-<?xml version="1.0"?>
-<robot xmlns:xacro="http://www.ros.org/wiki/xacro"  name="robot">
-	<!--<xacro:include filename="robot_core_lr.xacro"/>-->
-	<xacro:include filename="robot_core.xacro"/>
-	<xacro:include filename="gazebo_control.xacro"/>
-	<xacro:include filename="lidar.xacro"/>
-	<xacro:include filename="ros2_control.xacro"/>
-</robot>
+/home/vfran/billeagle_ws/bill_ws/src/bill/description/robot.urdf.xacro

File: bill_ws/install/bill/share/bill/description/robot_core.xacro (robot description, xacro)
@@ -1,194 +1 @@
-<?xml version="1.0"?>
-<robot xmlns:xacro="http://www.ros.org/wiki/xacro"  name="robot">
-    <!-- Main URDF file for Differential Drive Robot -->
-    <!-- Include general xacro files -->
-    <xacro:include filename="common.xacro"/>
-    <!-- Robot Variables -->
-    <xacro:property name="chassis_length" value="0.5"/>
-    <xacro:property name="chassis_width" value="0.3"/>
-    <xacro:property name="chassis_height" value="1.17"/>
-    <xacro:property name="chassis_mass" value="22.2"/>
-    <xacro:property name="wheel_radius" value="0.07"/>
-    <xacro:property name="wheel_thickness" value="0.05"/>
-    <xacro:property name="wheel_mass" value="0.2"/>
-    <xacro:property name="wheel_offset_x" value="0.2"/>
-    <xacro:property name="wheel_offset_y" value="${chassis_width/2 + wheel_thickness/2}"/>
-    <xacro:property name="wheel_offset_z" value="0.0"/>
-    <!-- Base Link -->
-    <link name="base_link"></link>
-    <!-- Base Footprint -->
-    <joint name="base_footprint_joint" type="fixed">
-        <parent link="base_link"/>
-        <child link="base_footprint"/>
-        <origin xyz="0 0 0" rpy="0 0 0"/>
-    </joint>
-    <link name="base_footprint"></link>
-    <!-- Chassis -->
-    <joint name="chassis_joint" type="fixed">
-        <parent link="base_link"/>
-        <child link="chassis_link"/>
-        <origin xyz="0 0 0"/>
-    </joint>
-    <link name="chassis_link">
-        <visual>
-            <origin xyz="0 0 ${chassis_height/2}"/>
-            <geometry>
-                <box size="${chassis_length} ${chassis_width} ${chassis_height}"/>
-            </geometry>
-            <material name="blue"/>
-        </visual>
-        <collision>
-            <origin xyz="0 0 ${chassis_height/2}"/>
-            <geometry>
-                <box size="${chassis_length} ${chassis_width} ${chassis_height}"/>
-            </geometry>
-        </collision>
-        <xacro:inertial_box mass="0.5" x="${chassis_length}" y="${chassis_width}" z="${chassis_height}">
-            <origin xyz="0 0 ${chassis_height/2}" rpy="0 0 0"/>
-        </xacro:inertial_box>
-    </link>
-    <!-- Front Left Wheel -->
-    <joint name="front_left_wheel_joint" type="continuous">
-        <parent link="base_link"/>
-        <child link="front_left_wheel"/>
-        <origin xyz="${wheel_offset_x} ${wheel_offset_y} 0" rpy="-${pi/2} 0 0" />
-        <axis xyz="0 0 1"/>
-    </joint>
-    <transmission name="front_left_wheel_trans">
-        <type>transmission_interface/SimpleTransmission</type>
-        <joint name="front_left_wheel_joint">
-            <hardwareInterface>hardware_interface/VelocityJointInterface</hardwareInterface>
-        </joint>
-        <actuator name="front_left_motor">
-            <hardwareInterface>hardware_interface/VelocityJointInterface</hardwareInterface>
-        </actuator>
-    </transmission>
-    <link name="front_left_wheel">
-        <visual>
-            <geometry>
-                <cylinder radius="${wheel_radius}" length="${wheel_thickness}"/>
-            </geometry>
-            <material name="white"/>
-        </visual>
-        <collision>
-            <geometry>
-                <sphere radius="${wheel_radius}"/>
-            </geometry>
-        </collision>
-        <xacro:inertial_cylinder mass="${wheel_mass}" length="${wheel_thickness}" radius="${wheel_radius}">
-            <origin xyz="0 0 0" rpy="0 0 0"/>
-        </xacro:inertial_cylinder>
-    </link>
-    <!-- Front Right Wheel -->
-    <joint name="front_right_wheel_joint" type="continuous">
-        <parent link="base_link"/>
-        <child link="front_right_wheel"/>
-        <origin xyz="${wheel_offset_x} ${-wheel_offset_y} 0" rpy="${pi/2} 0 0" />
-        <axis xyz="0 0 -1"/>
-    </joint>
-    <transmission name="front_right_wheel_trans">
-        <type>transmission_interface/SimpleTransmission</type>
-        <joint name="front_right_wheel_joint">
-            <hardwareInterface>hardware_interface/VelocityJointInterface</hardwareInterface>
-        </joint>
-        <actuator name="front_right_motor">
-            <hardwareInterface>hardware_interface/VelocityJointInterface</hardwareInterface>
-        </actuator>
-    </transmission>
-    <link name="front_right_wheel">
-        <visual>
-            <geometry>
-                <cylinder radius="${wheel_radius}" length="${wheel_thickness}"/>
-            </geometry>
-            <material name="white"/>
-        </visual>
-        <collision>
-            <geometry>
-                <sphere radius="${wheel_radius}"/>
-            </geometry>
-        </collision>
-        <xacro:inertial_cylinder mass="${wheel_mass}" length="${wheel_thickness}" radius="${wheel_radius}">
-            <origin xyz="0 0 0" rpy="0 0 0"/>
-        </xacro:inertial_cylinder>
-    </link>
-    <!-- Rear Left Wheel -->
-    <joint name="rear_left_wheel_joint" type="continuous">
-        <parent link="base_link"/>
-        <child link="rear_left_wheel"/>
-        <origin xyz="${-wheel_offset_x} ${wheel_offset_y} 0" rpy="-${pi/2} 0 0" />
-        <axis xyz="0 0 1"/>
-    </joint>
-    <transmission name="rear_left_wheel_trans">
-        <type>transmission_interface/SimpleTransmission</type>
-        <joint name="rear_left_wheel_joint">
-            <hardwareInterface>hardware_interface/VelocityJointInterface</hardwareInterface>
-        </joint>
-        <actuator name="rear_left_motor">
-            <hardwareInterface>hardware_interface/VelocityJointInterface</hardwareInterface>
-        </actuator>
-    </transmission>
-    <link name="rear_left_wheel">
-        <visual>
-            <geometry>
-                <cylinder radius="${wheel_radius}" length="${wheel_thickness}"/>
-            </geometry>
-            <material name="white"/>
-        </visual>
-        <collision>
-            <geometry>
-                <sphere radius="${wheel_radius}"/>
-            </geometry>
-        </collision>
-        <xacro:inertial_cylinder mass="${wheel_mass}" length="${wheel_thickness}" radius="${wheel_radius}">
-            <origin xyz="0 0 0" rpy="0 0 0"/>
-        </xacro:inertial_cylinder>
-    </link>
-    <!-- Rear Right Wheel -->
-    <joint name="rear_right_wheel_joint" type="continuous">
-        <parent link="base_link"/>
-        <child link="rear_right_wheel"/>
-        <origin xyz="${-wheel_offset_x} ${-wheel_offset_y} 0" rpy="${pi/2} 0 0" />
-        <axis xyz="0 0 -1"/>
-    </joint>
-    <transmission name="rear_right_wheel_trans">
-        <type>transmission_interface/SimpleTransmission</type>
-        <joint name="rear_right_wheel_joint">
-            <hardwareInterface>hardware_interface/VelocityJointInterface</hardwareInterface>
-        </joint>
-        <actuator name="rear_right_motor">
-            <hardwareInterface>hardware_interface/VelocityJointInterface</hardwareInterface>
-        </actuator>
-    </transmission>
-    <link name="rear_right_wheel">
-        <visual>
-            <geometry>
-                <cylinder radius="${wheel_radius}" length="${wheel_thickness}"/>
-            </geometry>
-            <material name="white"/>
-        </visual>
-        <collision>
-            <geometry>
-                <sphere radius="${wheel_radius}"/>
-            </geometry>
-        </collision>
-        <xacro:inertial_cylinder mass="${wheel_mass}" length="${wheel_thickness}" radius="${wheel_radius}">
-            <origin xyz="0 0 0" rpy="0 0 0"/>
-        </xacro:inertial_cylinder>
-    </link>
-    <!-- Gazebo -->
-    <gazebo reference="chassis_link">
-        <material>Gazebo/Blue</material>
-    </gazebo>
-    <gazebo reference="front_left_wheel">
-        <material>Gazebo/White</material>
-    </gazebo>
-    <gazebo reference="front_right_wheel">
-        <material>Gazebo/White</material>
-    </gazebo>
-    <gazebo reference="rear_left_wheel">
-        <material>Gazebo/White</material>
-    </gazebo>
-    <gazebo reference="rear_right_wheel">
-        <material>Gazebo/White</material>
-    </gazebo>
-</robot>
+/home/vfran/billeagle_ws/bill_ws/src/bill/description/robot_core.xacro

File: bill_ws/install/bill/share/bill/description/ros2_control.xacro (robot description, xacro)
@@ -1,47 +1 @@
-<?xml version="1.0"?>
-<robot xmlns:xacro="http://www.ros.org/wiki/xacro">
-    <ros2_control name="GazeboSystem" type="system">
-        <hardware>
-            <plugin>gazebo_ros2_control/GazeboSystem</plugin>
-        </hardware>
-        <!--Front wheels -->
-        <joint name="front_left_wheel_joint">
-            <command_interface name="velocity">
-                <param name="min">-10</param>
-                <param name="max">10</param>
-            </command_interface>
-            <state_interface name="velocity"/>
-            <state_interface name="position"/>
-        </joint>
-        <joint name="front_right_wheel_joint">
-            <command_interface name="velocity">
-                <param name="min">-10</param>
-                <param name="max">10</param>
-            </command_interface>
-            <state_interface name="velocity"/>
-            <state_interface name="position"/>
-        </joint>
-        <!-- Rear wheels -->
-        <joint name="rear_left_wheel_joint">
-            <command_interface name="velocity">
-                <param name="min">-10</param>
-                <param name="max">10</param>
-            </command_interface>
-            <state_interface name="velocity"/>
-            <state_interface name="position"/>
-        </joint>
-        <joint name="rear_left_wheel_trans">
-            <command_interface name="velocity">
-                <param name="min">-10</param>
-                <param name="max">10</param>
-            </command_interface>
-            <state_interface name="velocity"/>
-            <state_interface name="position"/>
-        </joint>
-    </ros2_control>
-    <gazebo>
-        <plugin name="gazebo_ros2_control" filename="libgazebo_ros2_control.so">
-            <parameters>$(find bill)/config/mecanum_drive_controller.yaml</parameters>
-        </plugin>
-    </gazebo>
-</robot>
+/home/vfran/billeagle_ws/bill_ws/src/bill/description/ros2_control.xacro

File: bill_ws/install/bill_description/share/bill_description/description/common.xacro (robot description, xacro)
@@ -1,60 +1 @@
-<?xml version="1.0"?>
-<robot xmlns:xacro="http://www.ros.org/wiki/xacro" >
-    <!-- This file contains the macros used across the URDF files -->
-    <!-- Inertial Macros -->
-    <!-- Inertial Sphere Macros -->
-    <xacro:macro name="inertial_sphere" params="mass radius *origin">
-        <inertial>
-            <xacro:insert_block name="origin"/>
-            <mass value="${mass}" />
-            <inertia ixx="${(2/5) * mass * (radius*radius)}" ixy="0.0" ixz="0.0"
-                    iyy="${(2/5) * mass * (radius*radius)}" iyz="0.0"
-                    izz="${(2/5) * mass * (radius*radius)}" />
-        </inertial>
-    </xacro:macro>
-    <!-- Inertial Box Macros -->
-    <xacro:macro name="inertial_box" params="mass x y z *origin">
-        <inertial>
-            <xacro:insert_block name="origin"/>
-            <mass value="${mass}" />
-            <inertia ixx="${(1/12) * mass * (y*y+z*z)}" ixy="0.0" ixz="0.0"
-                    iyy="${(1/12) * mass * (x*x+z*z)}" iyz="0.0"
-                    izz="${(1/12) * mass * (x*x+y*y)}" />
-        </inertial>
-    </xacro:macro>
-    <!-- Inertial Cylinder Macros -->
-    <xacro:macro name="inertial_cylinder" params="mass length radius *origin">
-        <inertial>
-            <xacro:insert_block name="origin"/>
-            <mass value="${mass}" />
-            <inertia ixx="${(1/12) * mass * (3*radius*radius + length*length)}" ixy="0.0" ixz="0.0"
-                    iyy="${(1/12) * mass * (3*radius*radius + length*length)}" iyz="0.0"
-                    izz="${(1/2) * mass * (radius*radius)}" />
-        </inertial>
-    </xacro:macro>
-    <!-- Material Macros -->
-    <material name="white">
-        <color rgba="1 1 1 1" />
-    </material>
-    <material name="orange">
-        <color rgba="1 0.3 0.1 1"/>
-    </material>
-    <material name="blue">
-        <color rgba="0.2 0.2 1 1"/>
-    </material>
-    <material name="black">
-        <color rgba="0 0 0 1"/>
-    </material>
-    <material name="red">
-        <color rgba="1 0 0 1"/>
-    </material>
-    <material name="grey">
-        <color rgba="0.631 0.631 0.631 1"/>
-    </material>
-    <material name="purple">
-        <color rgba="0.78 0.153 0.71 1"/>
-    </material>
-    <material name="green">
-        <color rgba="0.149 0.612 0.082 1"/>
-    </material>
-</robot>
+/home/vfran/billeagle_ws/bill_ws/src/bill_description/description/common.xacro

File: bill_ws/install/bill_description/share/bill_description/description/gazebo_control.xacro (robot description, xacro)
@@ -1,38 +1 @@
-<?xml version="1.0"?>
-<robot xmlns:xacro="http://www.ros.org/wiki/xacro">
-    <xacro:property name="wheel_radius" value="0.07"/>
-    <xacro:property name="wheel_thickness" value="0.05"/>
-    <xacro:property name="wheel_mass" value="0.2"/>
-    <xacro:property name="wheel_offset_x" value="0.2"/>
-    <xacro:property name="wheel_offset_y" value="${chassis_width/2 + wheel_thickness/2}"/>
-    <xacro:property name="wheel_offset_z" value="0.0"/>
-    <!-- Gazebo plugin for 4-wheel drive robots -->
-   <gazebo>
-      <plugin name="differential_drive_controller" filename="libgazebo_ros_diff_drive.so">
-        <!-- <ros>
-          <remapping>odom:=odom/unfiltered</remapping>
-        </ros> -->
-        <!-- <updateRate>100</updateRate> -->
-        <!-- Wheel Info -->
-        <num_wheel_pairs>2</num_wheel_pairs>
-        <left_joint>front_left_wheel_joint</left_joint>
-        <right_joint>front_right_wheel_joint</right_joint>
-        <left_joint>rear_left_wheel_joint</left_joint>
-        <right_joint>rear_right_wheel_joint</right_joint>
-        <wheel_separation>${wheel_offset_y*2}</wheel_separation>
-        <wheel_separation>${wheel_offset_y*2}</wheel_separation>
-        <wheel_diameter>${wheel_radius*2}</wheel_diameter>
-        <wheel_diameter>${wheel_radius*2}</wheel_diameter>
-        <!-- Limits -->
-        <max_wheel_torque>200</max_wheel_torque>
-        <max_wheel_acceleration>10.0</max_wheel_acceleration>
-        <!-- Frames -->
-        <odometry_frame>odom</odometry_frame>
-        <robot_base_frame>base_link</robot_base_frame>
-        <!-- Output -->
-        <publish_odom>true</publish_odom>
-        <publish_odom_tf>true</publish_odom_tf>
-        <publish_wheel_tf>true</publish_wheel_tf>
-      </plugin>
-    </gazebo>
-</robot>
+/home/vfran/billeagle_ws/bill_ws/src/bill_description/description/gazebo_control.xacro
