Commit message: mudando a cor do bill

File: bill_ws/src/bill_description/description/robot_core.xacro (robot description, xacro)
@@ -36,5 +36,5 @@
                 <box size="${chassis_length} ${chassis_width} ${chassis_height}"/>
             </geometry>
-            <material name="blue"/>
+            <material name="gray"/>
         </visual>
         <collision>
@@ -178,5 +178,5 @@
     <!-- Gazebo -->
     <gazebo reference="chassis_link">
-        <material>Gazebo/Blue</material>
+        <material>Gazebo/Gray</material>
     </gazebo>
     <gazebo reference="front_left_wheel">
